Commit message: ver.1.0

File: description/urdf/turtlebot3_waffle_pi.urdf.xacro (robot description, xacro)
@@ -174,5 +174,5 @@
   </link>
   <joint name="camera_rgb_joint" type="fixed">
-    <origin xyz="0.003 0.011 0.009" rpy="0 0 0"/>
+    <origin xyz="0.003 0.011 0.009" rpy="0 0.3 0"/>
     <parent link="camera_link"/>
     <child link="camera_rgb_frame"/>
